File: pathfinder.kicad_pcb (KiCad board)
At the start: 2 copper layers, 100 x 100 mm, 13 parts, among them SW4 SW_Push, U1 XIAO-RP2040-DIP

Commit message: redid pcb style and added another game
Parts:
- removed the SW4 at (122.5, 124.9)
- removed the SW4 at (152.5, 111.9)
- removed the SW4 at (182.5, 124.9)
- added  : LOGO, LOGO, F.Cu at (129.0, 104.0)
- added SW1: SW_Push, Button_Switch_Keyboard:SW_Cherry_MX_1.00u_PCB, F.Cu at (122.5, 124.9)
- added SW2: SW_Push, Button_Switch_Keyboard:SW_Cherry_MX_1.00u_PCB, F.Cu at (152.5, 111.9)
- added SW3: SW_Push, Button_Switch_Keyboard:SW_Cherry_MX_1.00u_PCB, F.Cu at (182.5, 124.9)
- moved D1 1.00 mm to (120.0, 91.0)
Connections:
- SW4 pad 1: (no net) -> button4
- SW4 pad 2: (no net) -> GND
Routing:
- net button2: track 146.6 -> 85.1 mm
- net button4: track 89.3 -> 107.4 mm
- net button3: track 82.2 -> 83.2 mm
- net button1: track 116.4 -> 115.5 mm
- net GND: track 226.2 -> 225.3 mm
Other:
- outline, holes or cut-outs redrawn
- board text added: "1"
- board text added: "2"
- board text added: "3"
- board text added: "4"
- board text added: "4 LEDs, 4 Buttons, What Games Can Be Made?"
- board text added: "By Guy Sandler"
